Commit message: Improve Isaac Sim simulation adding twist mux controller

File: nanosaur_isaac_sim/urdf/mecanum_drive.isaac.xacro (robot description, xacro)
@@ -2,5 +2,5 @@
 <robot name="mecanum_drive"
     xmlns:xacro="http://ros.org/wiki/xacro">
-    <xacro:macro name="mecanum_drive" params="parent wheelbase wheel_radius wheel_separation">
+    <xacro:macro name="mecanum_drive" params="parent name_space wheelbase wheel_radius wheel_separation">
         <isaacsim>
             <plugin name="JointStatePublisher">
@@ -8,4 +8,7 @@
             </plugin>
             <plugin name="MecanumDrive">
+                <!-- Namespace robot -->
+                <name_space>${name_space}</name_space>
+                <!-- joints definitions -->
                 <child_frame_id>${parent}</child_frame_id>
                 <front_left_joint>front_left_mecanum_joint</front_left_joint>
@@ -22,4 +25,6 @@
                 This element is optional, although it is recommended to be included with an appropriate value. The default value is 0.2m. -->
                 <wheel_radius>${wheel_radius}</wheel_radius>
+                <!-- Publish odometry -->
+                <publish_odom>false</publish_odom>
             </plugin>
         </isaacsim>

File: nanosaur_isaac_sim/urdf/nanosaur.isaac.xacro (robot description, xacro)
@@ -19,4 +19,5 @@
     <xacro:mecanum_drive
             parent="nanosaur_base"
+            name_space="$(arg robot_name)"
             wheelbase="${nanosaur_wheelbase}"
             wheel_radius="${mecanum_radius}"
